File: ATMega328 2016-09-04 SN74LV8154/kicad/simple.sch (KiCad schematic (older format))
At the start: 8 parts

Commit message: sn74lv8154
Parts:
- removed P?: SERIAL, symbol CONN_01X01
- added D?: LED2, symbol LED
- added R?: 47k, symbol R
- D?: value LED -> LED1
Connections:
- net GNDREF: now also D?.1 (K)
- net SERIAL: now reaches IC?.3 ((PCINT17/TXD)PD1)
- net at IC?.6 ((PCINT20/XCK/T0)PD4): now also R?.2
- new net: D?.2 (A), R?.1
Other:
- note added: "pay careful attention to power regulation,\ndecoupling inductor/capacitors, \nsignal input loading, etc"
- moved on the sheet: D?, R?
Changed lines of the file:
@@
 L R R?
 U 1 1 57CBC2EE
-P 8025 3800
-F 0 "R?" V 8105 3800 50  0000 C CNN
-F 1 "47k" V 8025 3800 50  0000 C CNN
-F 2 "" V 7955 3800 50  0000 C CNN
-F 3 "" H 8025 3800 50  0000 C CNN
-	1    8025 3800
+P 8250 3800
+F 0 "R?" V 8330 3800 50  0000 C CNN
+F 1 "47k" V 8250 3800 50  0000 C CNN
+F 2 "" V 8180 3800 50  0000 C CNN
+F 3 "" H 8250 3800 50  0000 C CNN
+	1    8250 3800
 	0    1    1    0
 $EndComp
 Wire Wire Line
-	7700 3800 7875 3800
+	7700 3800 8100 3800
 $Comp
 L LED D?
 U 1 1 57CBC449
-P 8375 3800
-F 0 "D?" H 8375 3900 50  0000 C CNN
-F 1 "LED" H 8375 3700 50  0000 C CNN
-F 2 "" H 8375 3800 50  0000 C CNN
-F 3 "" H 8375 3800 50  0000 C CNN
-	1    8375 3800
+P 8600 3800
+F 0 "D?" H 8600 3900 50  0000 C CNN
+F 1 "LED1" H 8600 3700 50  0000 C CNN
+F 2 "" H 8600 3800 50  0000 C CNN
+F 3 "" H 8600 3800 50  0000 C CNN
+	1    8600 3800
 	-1   0    0    1
 $EndComp
@@
 L GNDREF #PWR?
 U 1 1 57CBC4CA
-P 8575 3800
-F 0 "#PWR?" H 8575 3550 50  0001 C CNN
-F 1 "GNDREF" H 8575 3650 50  0001 C CNN
-F 2 "" H 8575 3800 50  0000 C CNN
-F 3 "" H 8575 3800 50  0000 C CNN
-	1    8575 3800
+P 8800 3800
+F 0 "#PWR?" H 8800 3550 50  0001 C CNN
+F 1 "GNDREF" H 8800 3650 50  0001 C CNN
+F 2 "" H 8800 3800 50  0000 C CNN
+F 3 "" H 8800 3800 50  0000 C CNN
+	1    8800 3800
 	1    0    0    -1
 $EndComp
@@
 Wire Wire Line
 	8275 2800 7700 2800
+Text Notes 3575 3775 0    60   ~ 0
+pay careful attention to power regulation,\ndecoupling inductor/capacitors, \nsignal input loading, etc
+Text Label 7700 3900 0    60   ~ 0
+SERIAL
 $Comp
-L CONN_01X01 P?
-U 1 1 57CBD2EA
-P 8050 4100
-F 0 "P?" H 8050 4200 50  0000 C CNN
-F 1 "SERIAL" V 8150 4100 50  0000 C CNN
-F 2 "" H 8050 4100 50  0000 C CNN
-F 3 "" H 8050 4100 50  0000 C CNN
-	1    8050 4100
+L R R?
+U 1 1 57CD9617
+P 8250 4200
+F 0 "R?" V 8330 4200 50  0000 C CNN
+F 1 "47k" V 8250 4200 50  0000 C CNN
+F 2 "" V 8180 4200 50  0000 C CNN
+F 3 "" H 8250 4200 50  0000 C CNN
+	1    8250 4200
+	0    1    1    0
+$EndComp
+$Comp
+L LED D?
+U 1 1 57CD961D
+P 8600 4200
+F 0 "D?" H 8600 4300 50  0000 C CNN
+F 1 "LED2" H 8600 4100 50  0000 C CNN
+F 2 "" H 8600 4200 50  0000 C CNN
+F 3 "" H 8600 4200 50  0000 C CNN
+	1    8600 4200
+	-1   0    0    1
+$EndComp
+$Comp
+L GNDREF #PWR?
+U 1 1 57CD9623
+P 8800 4200
+F 0 "#PWR?" H 8800 3950 50  0001 C CNN
+F 1 "GNDREF" H 8800 4050 50  0001 C CNN
+F 2 "" H 8800 4200 50  0000 C CNN
+F 3 "" H 8800 4200 50  0000 C CNN
+	1    8800 4200
 	1    0    0    -1
 $EndComp
 Wire Wire Line
-	7700 3900 7825 3900
-Wire Wire Line
-	7825 3900 7825 4100
-Wire Wire Line
-	7825 4100 7850 4100
+	8100 4200 7700 4200
 $EndSCHEMATC
